File: strut.kicad_pcb (KiCad board)
At the start: 2 copper layers, 262.2 x 37.5 mm, 2 parts

Commit message: Exported step files
Parts:
- removed REF** (x2): Spoke_Connector, local:Spoke_Connector
- added J1: Left, local:Spoke_Connector, B.Cu at (81.3, 148.0)
- added J2: Right, local:Spoke_Connector, F.Cu at (338.7, 148.0)
Other:
- board size 262.2 x 37.5 mm -> 296.3 x 48.5 mm

Commit message: Now with the proper angles
Parts:
- moved J1 10.0 mm to (91.3, 148.0)
- moved J2 10.0 mm to (328.7, 148.0)
Other:
- board size 296.3 x 48.5 mm -> 276.3 x 44.8 mm
